File: tmp_30.brd (EAGLE design)
At the start: 31.8 x 81.7 mm, 0 parts

Commit message: union signal
Changed lines of the file:
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@@
 <setting verticaltext="up"/>
 </settings>
-<grid distance="0.05" unitdist="inch" unit="inch" style="lines" multiple="1" display="no" altdistance="0.025" altunitdist="inch" altunit="inch"/>
+<grid distance="0.05" unitdist="inch" unit="mm" style="lines" multiple="1" display="no" altdistance="0.025" altunitdist="inch" altunit="mm"/>
 <layers>
 <layer number="1" name="Top" color="4" fill="1" visible="yes" active="yes"/>
@@
 <board>
 <plain>
-<wire x1="0" y1="0" x2="31.78" y2="0" width="0" layer="20"/>
-<wire x1="31.78" y1="0" x2="31.78" y2="81.66" width="0" layer="20"/>
-<wire x1="31.78" y1="81.66" x2="0" y2="81.66" width="0" layer="20"/>
-<wire x1="0" y1="81.66" x2="0" y2="0" width="0" layer="20"/>
+<wire x1="0" y1="87.76" x2="31.78" y2="87.76" width="0" layer="20"/>
+<wire x1="31.78" y1="87.76" x2="31.78" y2="169.42" width="0" layer="20"/>
+<wire x1="31.78" y1="169.42" x2="0" y2="169.42" width="0" layer="20"/>
+<wire x1="0" y1="169.42" x2="0" y2="87.76" width="0" layer="20"/>
 </plain>
 <attributes>
@@
 </class>
 </classes>
-<designrules name="default">
+<designrules name="default *">
 <description language="de">&lt;b&gt;EAGLE Design Rules&lt;/b&gt;
 &lt;p&gt;
@@
 <param name="mtCopper" value="0.035mm 0.035mm 0.035mm 0.035mm 0.035mm 0.035mm 0.035mm 0.035mm 0.035mm 0.035mm 0.035mm 0.035mm 0.035mm 0.035mm 0.035mm 0.035mm"/>
 <param name="mtIsolate" value="1.5mm 0.15mm 0.2mm 0.15mm 0.2mm 0.15mm 0.2mm 0.15mm 0.2mm 0.15mm 0.2mm 0.15mm 0.2mm 0.15mm 0.2mm"/>
-<param name="mdWireWire" value="8mil"/>
-<param name="mdWirePad" value="8mil"/>
+<param name="mdWireWire" value="12mil"/>
+<param name="mdWirePad" value="10mil"/>
 <param name="mdWireVia" value="8mil"/>
 <param name="mdPadPad" value="8mil"/>
